File: KBD.kicad_pcb (KiCad board)
At the start: 2 copper layers, 97.5 x 91.7 mm, 39 parts, among them J1 Conn_01x07, J2 Conn_01x07, SW1 SW_Push, SW10 SW_Push, SW11 SW_Push, SW12 SW_Push, SW13 SW_Push, SW14 SW_Push, SW15 SW_Push, SW16 SW_Push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

Commit message: bbbbbb2
Parts:
- added D20: WS2812B, LED_SMD:LED_WS2812B_PLCC4_5.0x5.0mm_P3.2mm, B.Cu at (184.1, 95.4)
Connections:
- D19 pad 2: unconnected-(D19-DOUT-Pad2) -> Net-(D19-DOUT)
Routing:
- net 5V: track 26.2 -> 33.3 mm
- net Net-(D19-DOUT): track 0.00 -> 3.87 mm, vias 0 -> 1
- net Led_In: track 25.5 -> 28.7 mm
- net Column_3: track 119.2 -> 116.2 mm
- net 0V: track 27.0 -> 28.7 mm
- net Row_2: track 117.6 -> 116.1 mm
- net Row_3: track 93.6 -> 92.2 mm
- net Row_4: track 49.6 -> 48.4 mm
- net Column_2: track 124.9 -> 125.9 mm
- net Column_1: track 138.3 -> 137.2 mm
- net Column_5: track 81.8 -> 81.3 mm
- net unconnected-(D19-DOUT-Pad2): vias 1 -> 0

Commit message: TRRS version
Parts:
- added R1: 4.7k, Resistor_SMD:R_0805_2012Metric, F.Cu at (160.7, 126.8)
- added R2: 4.7k, Resistor_SMD:R_0805_2012Metric, F.Cu at (160.7, 129.8)
- added TRRS1: ~, SparkFun-Connectors:AUDIO-JACK-TRRS-SMD, F.Cu at (167.3, 125.0)
Connections:
- J1 pad 5: Led_In -> SDA
- J1 pad 6: Column_1 -> SCL
- J1 pad 7: unconnected-(J1-Pin_7-Pad7) -> Column_1
- J2 pad 1: Column_2 -> Led_In
- J2 pad 2: Column_3 -> Column_2
- J2 pad 3: Column_4 -> Column_3
- J2 pad 4: Column_5 -> Column_4
- J2 pad 5: unconnected-(J2-Pin_5-Pad5) -> Column_5
Routing:
- net Row_1: track 133.8 -> 80.5 mm
- net Column_1: track 137.2 -> 97.8 mm
- net Row_2: track 116.1 -> 76.9 mm
- net Column_3: track 116.2 -> 77.4 mm
- net Led_In: track 28.7 -> 0.49 mm
- net Row_3: track 92.2 -> 68.8 mm
- net Column_2: track 125.9 -> 104.0 mm
- net Column_5: track 81.3 -> 66.7 mm
- net Column_4: track 78.3 -> 66.6 mm

Commit message: led not routed, else is done
Parts:
- removed TRRS1: ~, SparkFun-Connectors:AUDIO-JACK-TRRS-SMD
- added J1: Conn_01x07, Connector_Hirose:Hirose_DF13-07P-1.25DS_1x07_P1.25mm_Horizontal, B.Cu at (157.4, 93.8)
- added J2: Conn_01x07, Connector_Hirose:Hirose_DF13-07P-1.25DS_1x07_P1.25mm_Horizontal, B.Cu at (175.3, 107.0)
- added J3: AudioJack4, Connector_Audio:Jack_3.5mm_PJ320D_Horizontal, F.Cu at (171.7, 114.3)
- added J3: AudioJack4, Connector_Audio:Jack_3.5mm_PJ320D_Horizontal, B.Cu at (171.7, 114.3)
- added SW19: SW_DIP_x01, Button_Switch_THT:SW_DIP_SPSTx01_Slide_6.7x4.1mm_W7.62mm_P2.54mm_LowProfile, F.Cu at (189.3, 100.5)
- added TP1: TestPoint, TestPoint:TestPoint_THTPad_2.0x2.0mm_Drill1.0mm, F.Cu at (177.0, 102.9)
- added TP2: TestPoint, TestPoint:TestPoint_THTPad_2.0x2.0mm_Drill1.0mm, F.Cu at (177.0, 99.7)
- moved R2 27.1 mm to (177.3, 108.3), turned to -105 degrees
- moved R1 25.3 mm to (179.2, 109.6), turned to -105 degrees
- moved D18 6.58 mm to (180.4, 105.4)
- moved SW17 2.11 mm to (204.0, 117.4)
- moved SW16 2.11 mm to (220.4, 123.5)
- moved SW18 2.11 mm to (187.3, 112.1)
- moved D16 1.64 mm to (211.1, 123.6)
- moved D17 1.46 mm to (194.6, 118.4)
Connections:
- R1 pad 2: SCL -> SDA
Routing:
- net Column_1: track 97.8 -> 156.4 mm
- net Column_3: track 77.4 -> 127.9 mm
- net Row_1: track 80.5 -> 129.4 mm
- net Column_2: track 104.0 -> 150.3 mm
- net Row_4: track 48.4 -> 88.4 mm
- net SDA: track 0.00 -> 36.0 mm, vias 0 -> 2
- net Row_2: track 76.9 -> 111.0 mm, vias 5 -> 6
- net SCL: track 0.00 -> 31.3 mm, vias 0 -> 2
- net Column_5: track 66.7 -> 97.4 mm
- net Led_In: track 0.49 -> 30.3 mm
- net Column_4: track 66.6 -> 94.0 mm
- net 5V: track 33.3 -> 56.0 mm, vias 1 -> 3
- net Row_3: track 68.8 -> 90.6 mm
- net Bat+: track 0.00 -> 13.3 mm
- net MCU_Bat+: track 0.00 -> 5.00 mm
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Other:
- board size 97.5 x 91.7 mm -> 97.5 x 93 mm

Commit message: routing chaos
Parts:
- removed the SW19 at (189.3, 100.5)
- added SW19: SW_DIP_x04, Button_Switch_SMD:SW_DIP_SPSTx04_Slide_Copal_CHS-04A_W5.08mm_P1.27mm_JPin, F.Cu at (184.0, 98.6)
- added SW19: SW_DIP_x04, Button_Switch_SMD:SW_DIP_SPSTx04_Slide_Copal_CHS-04A_W5.08mm_P1.27mm_JPin, B.Cu at (184.0, 98.6)
- added TP3: TestPoint, TestPoint:TestPoint_Pad_1.0x1.0mm, B.Cu at (160.8, 112.9)
- added TP4: TestPoint, TestPoint:TestPoint_Pad_1.0x1.0mm, B.Cu at (163.6, 112.4)
- added TP5: TestPoint, TestPoint:TestPoint_Pad_1.0x1.0mm, B.Cu at (162.2, 112.6)
- TP1, TP2: footprint TestPoint:TestPoint_THTPad_2.0x2.0mm_Drill1.0mm -> TestPoint:TestPoint_THTPad_1.5x1.5mm_Drill0.7mm
- moved D20 5.65 mm to (179.6, 92.1)
- moved D19 5.37 mm to (178.3, 92.1)
- moved TP1 2.92 mm to (177.2, 99.9)
- moved TP2 2.42 mm to (177.2, 102.1)
Connections:
- D19 pad 4: Led_In -> LED_IN
- J2 pad 1: Led_In -> Column_2 (x2)
- J2 pad 2: Column_2 -> Column_3 (x2)
- J2 pad 3: Column_3 -> Column_4 (x2)
- J2 pad 4: Column_4 -> Column_5 (x2)
- J2 pad 5: Column_5 -> 3.3V (x2)
- J3 pad S: 5V -> I2CPullUp (x2)
- R1 pad 1: 5V -> I2CPullUp
- R2 pad 1: 5V -> I2CPullUp
Routing:
- net 3.3V: track 0.00 -> 47.5 mm, vias 0 -> 1
- net I2CPullUp: track 0.00 -> 34.5 mm, vias 0 -> 2
- net Led_In: track 30.3 -> 0.00 mm, vias 1 -> 0
- net 0V: track 33.2 -> 59.7 mm
- net Bat+: track 13.3 -> 0.00 mm, vias 0 -> 1
- net Row_3: track 90.6 -> 101.3 mm
- net Row_1: track 129.4 -> 137.6 mm
- net Column_2: track 150.3 -> 142.8 mm
- net MCU_Bat+: track 5.00 -> 0.00 mm, vias 0 -> 1
- net Column_5: track 97.4 -> 101.7 mm
- net Net-(D19-DOUT): track 3.87 -> 0.00 mm
- net Column_3: track 127.9 -> 124.4 mm
- net 5V: track 56.0 -> 59.2 mm
- net Column_4: track 94.0 -> 97.1 mm
- net SDA: track 36.0 -> 35.1 mm
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