File: KBD.kicad_sch (KiCad schematic)
At the start: 50 parts, among them J1 Conn_01x07, J2 Conn_01x07, J3 AudioJack4, SW1 SW_Push, SW10 SW_Push, SW11 SW_Push, SW12 SW_Push, SW13 SW_Push, SW14 SW_Push, SW15 SW_Push, SW16 SW_Push, SW17 SW_Push, SW18 SW_Push, SW19 SW_DIP_x04, SW2 SW_Push, SW3 SW_Push, SW4 SW_Push, SW5 SW_Push, SW6 SW_Push, SW7 SW_Push, SW8 SW_Push, SW9 SW_Push, U1 SeeeduinoXIAO

Commit message: Almost done
Connections:
- net 5V: no longer D19.1 (VDD), D20.1 (VDD)
- net LED_IN: now also D20.4 (DIN)
- net LED_PWR: now also D19.1 (VDD), D20.1 (VDD)
- net at D19.2 (DOUT): no longer D20.4 (DIN)
Changed lines of the file:
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@@
     (stroke (width 0) (type default))
   )
-  (global_label "5V" (shape input) (at 119.38 85.09 90) (fields_autoplaced)
-    (effects (font (size 1.27 1.27)) (justify left))
-    (property "Intersheetrefs" "${INTERSHEET_REFS}" (at 119.38 79.8861 90)
+  (global_label "LED_PWR" (shape input) (at 109.22 90.17 90) (fields_autoplaced)
+    (effects (font (size 1.27 1.27)) (justify left))
+    (property "Intersheetrefs" "${INTERSHEET_REFS}" (at 109.22 78.8581 90)
       (effects (font (size 1.27 1.27)) (justify left) hide)
     )
@@
     )
   )
-  (global_label "0V" (shape input) (at 134.62 100.33 270) (fields_autoplaced)
-    (effects (font (size 1.27 1.27)) (justify right))
-    (property "Intersheetrefs" "${INTERSHEET_REFS}" (at 134.62 105.5339 90)
+  (global_label "0V" (shape input) (at 139.7 105.41 270) (fields_autoplaced)
+    (effects (font (size 1.27 1.27)) (justify right))
+    (property "Intersheetrefs" "${INTERSHEET_REFS}" (at 139.7 110.6139 90)
       (effects (font (size 1.27 1.27)) (justify right) hide)
     )
@@
     )
   )
+  (global_label "LED_IN" (shape input) (at 132.08 97.79 180) (fields_autoplaced)
+    (effects (font (size 1.27 1.27)) (justify right))
+    (property "Intersheetrefs" "${INTERSHEET_REFS}" (at 122.8242 97.79 0)
+      (effects (font (size 1.27 1.27)) (justify right) hide)
+    )
+  )
   (global_label "MCU_Bat+" (shape passive) (at 139.7 130.81 0) (fields_autoplaced)
     (effects (font (size 1.27 1.27)) (justify left))
@@
     )
   )
-  (global_label "LED_IN" (shape input) (at 111.76 92.71 180) (fields_autoplaced)
-    (effects (font (size 1.27 1.27)) (justify right))
-    (property "Intersheetrefs" "${INTERSHEET_REFS}" (at 102.5042 92.71 0)
+  (global_label "LED_IN" (shape input) (at 101.6 97.79 180) (fields_autoplaced)
+    (effects (font (size 1.27 1.27)) (justify right))
+    (property "Intersheetrefs" "${INTERSHEET_REFS}" (at 92.3442 97.79 0)
       (effects (font (size 1.27 1.27)) (justify right) hide)
     )
@@
     )
   )
-  (global_label "5V" (shape input) (at 134.62 85.09 90) (fields_autoplaced)
-    (effects (font (size 1.27 1.27)) (justify left))
-    (property "Intersheetrefs" "${INTERSHEET_REFS}" (at 134.62 79.8861 90)
+  (global_label "LED_PWR" (shape input) (at 139.7 90.17 90) (fields_autoplaced)
+    (effects (font (size 1.27 1.27)) (justify left))
+    (property "Intersheetrefs" "${INTERSHEET_REFS}" (at 139.7 78.8581 90)
       (effects (font (size 1.27 1.27)) (justify left) hide)
     )
@@
     )
   )
-  (global_label "0V" (shape input) (at 119.38 100.33 270) (fields_autoplaced)
-    (effects (font (size 1.27 1.27)) (justify right))
-    (property "Intersheetrefs" "${INTERSHEET_REFS}" (at 119.38 105.5339 90)
+  (global_label "0V" (shape input) (at 109.22 105.41 270) (fields_autoplaced)
+    (effects (font (size 1.27 1.27)) (justify right))
+    (property "Intersheetrefs" "${INTERSHEET_REFS}" (at 109.22 110.6139 90)
       (effects (font (size 1.27 1.27)) (justify right) hide)
     )
@@
     )
   )
-  (symbol (lib_id "LED:WS2812B") (at 134.62 92.71 0) (unit 1)
-    (in_bom yes) (on_board yes) (dnp no) (fields_autoplaced)
-    (property "Reference" "D20" (at 146.05 88.8239 0)
-      (effects (font (size 1.27 1.27)) hide)
-    )
-    (property "Value" "WS2812B" (at 146.05 91.3639 0)
-      (effects (font (size 1.27 1.27)) hide)
-    )
-    (property "Footprint" "LED_SMD:LED_WS2812B_PLCC4_5.0x5.0mm_P3.2mm" (at 135.89 100.33 0)
+  (symbol (lib_id "LED:WS2812B") (at 139.7 97.79 0) (unit 1)
+    (in_bom yes) (on_board yes) (dnp no) (fields_autoplaced)
+    (property "Reference" "D20" (at 151.13 93.9039 0)
+      (effects (font (size 1.27 1.27)) hide)
+    )
+    (property "Value" "WS2812B" (at 151.13 96.4439 0)
+      (effects (font (size 1.27 1.27)) hide)
+    )
+    (property "Footprint" "LED_SMD:LED_WS2812B_PLCC4_5.0x5.0mm_P3.2mm" (at 140.97 105.41 0)
       (effects (font (size 1.27 1.27)) (justify left top) hide)
     )
-    (property "Datasheet" "https://cdn-shop.adafruit.com/datasheets/WS2812B.pdf" (at 137.16 102.235 0)
+    (property "Datasheet" "https://cdn-shop.adafruit.com/datasheets/WS2812B.pdf" (at 142.24 107.315 0)
       (effects (font (size 1.27 1.27)) (justify left top) hide)
     )
@@
     )
   )
-  (symbol (lib_id "LED:WS2812B") (at 119.38 92.71 0) (unit 1)
-    (in_bom yes) (on_board yes) (dnp no) (fields_autoplaced)
-    (property "Reference" "D19" (at 130.81 88.8239 0)
-      (effects (font (size 1.27 1.27)) hide)
-    )
-    (property "Value" "WS2812B" (at 130.81 91.3639 0)
-      (effects (font (size 1.27 1.27)) hide)
-    )
-    (property "Footprint" "LED_SMD:LED_WS2812B_PLCC4_5.0x5.0mm_P3.2mm" (at 120.65 100.33 0)
+  (symbol (lib_id "LED:WS2812B") (at 109.22 97.79 0) (unit 1)
+    (in_bom yes) (on_board yes) (dnp no) (fields_autoplaced)
+    (property "Reference" "D19" (at 120.65 93.9039 0)
+      (effects (font (size 1.27 1.27)) hide)
+    )
+    (property "Value" "WS2812B" (at 120.65 96.4439 0)
+      (effects (font (size 1.27 1.27)) hide)
+    )
+    (property "Footprint" "LED_SMD:LED_WS2812B_PLCC4_5.0x5.0mm_P3.2mm" (at 110.49 105.41 0)
       (effects (font (size 1.27 1.27)) (justify left top) hide)
     )
-    (property "Datasheet" "https://cdn-shop.adafruit.com/datasheets/WS2812B.pdf" (at 121.92 102.235 0)
+    (property "Datasheet" "https://cdn-shop.adafruit.com/datasheets/WS2812B.pdf" (at 111.76 107.315 0)
       (effects (font (size 1.27 1.27)) (justify left top) hide)
     )
